File: dimmer.kicad_sch (KiCad schematic)
At the start: 38 parts

Commit message: Switch to buck & go to production!
Parts:
- removed U1: (no value), symbol Regulator_Linear:AZ1084-5.0
- added C10, C11: 10u, Capacitor_SMD:C_0402_1005Metric, symbol Device:C_Small
- added C12: 100n, Capacitor_SMD:C_0402_1005Metric, symbol Device:C_Small
- added L1: 15uH 750mA, Inductor_SMD:L_Bourns-SRN4018, symbol Device:L_Ferrite
- added R15: 51k, Resistor_SMD:R_0402_1005Metric, symbol Device:R_Small
- added R16: 10k, Resistor_SMD:R_0402_1005Metric, symbol Device:R_Small
- added U1: RY8310, Package_TO_SOT_SMD:TSOT-23-6, symbol Regulator_Switching:LM2734Y
- C1: value (none) -> 10u 50V; footprint (none) -> Capacitor_SMD:C_0805_2012Metric
- C2, C4, C6: value (none) -> 10u; footprint (none) -> Capacitor_SMD:C_0402_1005Metric
- C3, C5, C7, C8, C9: value (none) -> 100n; footprint (none) -> Capacitor_SMD:C_0402_1005Metric
- J1, J2: value (none) -> Conn_01x02; footprint (none) -> Connector_PinHeader_2.54mm:PinHeader_1x02_P2.54mm_Vertical
- J3: value (none) -> Conn_01x05; footprint (none) -> Connector_PinHeader_1.27mm:PinHeader_1x05_P1.27mm_Vertical
- JP1: value (none) -> SolderJumper_2_Open; footprint (none) -> Jumper:SolderJumper-2_P1.3mm_Open_TrianglePad1.0x1.5mm
- LOGO1: value (none) -> Logo_Open_Hardware_Small; footprint (none) -> Symbol:OSHW-Logo2_7.3x6mm_SilkScreen
- Q1, Q2, Q3, Q4, Q5: value (none) -> HY1503C1; footprint (none) -> Library:DFN-8-1EP_3x3mm_P0.65mm_EP2x2.4mm
- R1: value (none) -> 1k; footprint (none) -> Resistor_SMD:R_0402_1005Metric
- R10, R11, R12, R13, R9: value (none) -> 100; footprint (none) -> Resistor_SMD:R_0402_1005Metric
- R14: value (none) -> 2.4k; footprint (none) -> Resistor_SMD:R_0402_1005Metric
- R2, R3, R4, R5, R6, R7, R8: value (none) -> 10k; footprint (none) -> Resistor_SMD:R_0402_1005Metric
- U2: value (none) -> AMS1117-3.3; footprint (none) -> Package_TO_SOT_SMD:SOT-223-3_TabPin2
- U3: value (none) -> ESP-12F; footprint (none) -> RF_Module:ESP-12E
- U4: value (none) -> SN74AVC8T245PW; footprint (none) -> Package_SO:TSSOP-24_4.4x7.8mm_P0.65mm
Connections:
- net +5V: now also C10.1, C11.1, L1.2, R15.1; no longer C3.1
- net GND: now also C10.2, C11.2, R16.2, U1.2 (GND)
- net VCC: now also C3.1, U1.4 (EN), U1.5 (VIN)
- new net: C12.2, L1.1, U1.6 (SW)
- new net: C12.1, U1.1 (BOOST)
- new net: R15.2, R16.1, U1.3 (FB)
Other:
- moved on the sheet: C2, C4, U2

Commit message: Simplify design
Parts:
- removed C8, C9: 100n, Capacitor_SMD:C_0402_1005Metric, symbol Device:C_Small
- removed J3: Conn_01x05, Connector_PinHeader_1.27mm:PinHeader_1x05_P1.27mm_Vertical, symbol Connector_Generic:Conn_01x05
- removed U4: SN74AVC8T245PW, Package_SO:TSSOP-24_4.4x7.8mm_P0.65mm, symbol Logic_LevelTranslator:SN74AVC8T245PW
- added Q10, Q6, Q7, Q8, Q9: WNM2030, Package_TO_SOT_SMD:SOT-723, symbol Device:Q_NMOS_GSD
- J1: footprint Connector_PinHeader_2.54mm:PinHeader_1x02_P2.54mm_Vertical -> Connector_Wire:SolderWire-1sqmm_1x02_P5.4mm_D1.4mm_OD2.7mm
- J4: value (none) -> Conn_01x06; footprint (none) -> Library:PinHeader_1x06_P2.54mm_Horizontal
- R10, R11, R12, R13, R9: value 100 -> 2.4k; LCSC C25076 -> C25882
- R16, R2, R3, R4, R5, R6, R7, R8: LCSC C25076 -> C25744
Connections:
- net +3V3 is gone; now on net +3.3V: C4.1, C6.1, C7.1, R14.1, R2.1, R3.1, U2.2 (VO), U3.8 (VCC)
- net +5V: now also R10.1, R11.1, R12.1, R13.1, R9.1
- net CH0_D: now also R4.2, U3.17 (GPIO2), Q6.1 (G); no longer U3.4 (GPIO16)
- net CH1_D: now also R5.2, U3.7 (GPIO13), Q7.1 (G); no longer U3.5 (GPIO14)
- net CH2_D: now also R6.2, Q8.1 (G)
- net CH3_D: now also R7.2, U3.4 (GPIO16), Q9.1 (G); no longer U3.7 (GPIO13)
- net CH4_D: now also R8.2, U3.5 (GPIO14), Q10.1 (G); no longer U3.17 (GPIO2)
- net GND: now also Q10.2 (S), Q6.2 (S), Q7.2 (S), Q8.2 (S), Q9.2 (S); no longer R4.2, R5.2, R6.2, R7.2, R8.2
- net +3.3V: now reaches R6.1
- net +3.3V: now also R4.1, R5.1, R7.1, R8.1; no longer R11.1
- net at Q3.2 (G), R11.2: now also Q8.3 (D)
- net at Q2.2 (G), R10.2: now also Q7.3 (D)
- net at Q5.2 (G), R13.2: now also Q10.3 (D)
- net at Q4.2 (G), R12.2: now also Q9.3 (D)
- net at Q1.2 (G), R9.2: now also Q6.3 (D)
- no-connect marks 15 -> 9
Other:
- moved on the sheet: J4, Q1, Q2, Q3, Q4, Q5, R4, R5, R6, R7, R8

Commit message: reannotate
Parts:
- renumbered C5 to C1, C1 to C10, C7 to C2, C6 to C3, C10 to C4, C11 to C5, C12 to C6, C2 to C7, C3 to C8, C4 to C9, J2 to J1, J1 to J2, J4 to J3, Q10 to Q1, Q1 to Q10, Q9 to Q2, Q8 to Q3, Q7 to Q4, Q6 to Q5, Q5 to Q6, Q4 to Q7, Q3 to Q8, Q2 to Q9, R2 to R1, R5 to R10, R4 to R11, R13 to R12, R12 to R13, R11 to R14, R10 to R15, R9 to R16, R3 to R2, R14 to R3, R1 to R4, R15 to R5, R16 to R6, R8 to R7, R7 to R8, R6 to R9, U3 to U1, U1 to U3
